File: hardware/pcb/hauptplatine/tools/routing/final_nach_maze_vor_polish.kicad_pcb (KiCad board)
At the start: 4 copper layers, 41 x 97 mm, 153 parts, among them J1 SJ-43504-SMT-TR, J20 FH12-30S-0.5SH(55), J21 503480-0600, J4 microSD, J6 USB, Q1 PMV48XPA2R, Q10 2N7002T, Q11 2N7002T, Q20 2N7002T, SW1 B3U-3000P, U10 MCP73871, U12 TUSB320LAI, U15 ESP32-S31-WROOM-1-N16R16V, U16 TPS22948, U17 CS43131-CNZR, U20 TPS61023DRL, U21 TPS2553DRV, U22 MAX17048G+T10, U3 D5V0L2B3T-7, U30 PCA9306DCUR, U31 SN74AXC1T45DRL, U32 SN74AXC1T45DRL, U33 SN74AXC1T45DRL, U34 TLV75518PDRV, U4 TLV75733PDRV, U5 PE1605C4A6, X1 22.5792MHz, X2 24.576MHz

Commit message: Hauptplatine geroutet: Doku, Maße und Problemliste aktualisiert
Co-Authored-By: Claude Sonnet 5.5 <noreply@anthropic.com>
Claude-Session: https://claude.ai/code/session_01JifvE6gExGmwsJWDpfRrrS
Connections:
- D10 pad 2: unconnected-(D10-NC_2-Pad2) -> (no net)
- J1 pad 6: unconnected-(J1-NC_6-Pad6) -> (no net)
- J20 pad 13: unconnected-(J20-NC_13-Pad13) -> (no net)
- J21 pad 6: unconnected-(J21-NC_6-Pad6) -> (no net)
- J6 pad A8: unconnected-(J6-NC_A8-PadA8) -> (no net)
- J6 pad B8: unconnected-(J6-NC_B8-PadB8) -> (no net)
- U12 pad 3: unconnected-(U12-NC_3-Pad3) -> (no net)
- U15 pad 26: unconnected-(U15-NC_26-Pad26) -> (no net)
- U15 pad 29: unconnected-(U15-NC_29-Pad29) -> (no net)
- U15 pad 30: unconnected-(U15-NC_30-Pad30) -> (no net)
- U15 pad 31: unconnected-(U15-NC_31-Pad31) -> (no net)
- U15 pad 32: unconnected-(U15-NC_32-Pad32) -> (no net)
- U15 pad 33: unconnected-(U15-NC_33-Pad33) -> (no net)
- U15 pad 34: unconnected-(U15-NC_34-Pad34) -> (no net)
- U15 pad 35: unconnected-(U15-NC_35-Pad35) -> (no net)
- U15 pad 38: unconnected-(U15-NC_38-Pad38) -> (no net)
- U15 pad 39: unconnected-(U15-NC_39-Pad39) -> (no net)
- U15 pad 42: unconnected-(U15-NC_42-Pad42) -> (no net)
- U15 pad 60: unconnected-(U15-NC_60-Pad60) -> (no net)
- U15 pad 61: unconnected-(U15-NC_61-Pad61) -> (no net)
- U16 pad 4: unconnected-(U16-NC_4-Pad4) -> (no net)
- U17 pad 12: unconnected-(U17-NC_12-Pad12) -> (no net)
- U17 pad 15: unconnected-(U17-NC_15-Pad15) -> (no net)
- U17 pad 29: unconnected-(U17-NC_29-Pad29) -> (no net)
- U17 pad 3: unconnected-(U17-NC_3-Pad3) -> (no net)
- U17 pad 32: unconnected-(U17-NC_32-Pad32) -> (no net)
- U17 pad 33: unconnected-(U17-NC_33-Pad33) -> (no net)
- U17 pad 40: unconnected-(U17-NC_40-Pad40) -> (no net)
- U34 pad 2: unconnected-(U34-NC_2-Pad2) -> (no net)
- U34 pad 5: unconnected-(U34-NC_5-Pad5) -> (no net)
- U4 pad 2: unconnected-(U4-NC_2-Pad2) -> (no net)
- U4 pad 5: unconnected-(U4-NC_5-Pad5) -> (no net)
Changed lines of the file:
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@@
 	(net 103 "LCD_IM0")
 	(net 104 "LCD_PWR_EN")
-	(net 105 "unconnected-(U16-NC_4-Pad4)")
-	(net 106 "unconnected-(U4-NC_2-Pad2)")
-	(net 107 "unconnected-(U4-NC_5-Pad5)")
-	(net 108 "unconnected-(J21-NC_6-Pad6)")
-	(net 109 "unconnected-(J20-NC_13-Pad13)")
-	(net 110 "unconnected-(U12-NC_3-Pad3)")
-	(net 111 "unconnected-(D10-NC_2-Pad2)")
-	(net 112 "unconnected-(J1-NC_6-Pad6)")
-	(net 113 "unconnected-(U34-NC_2-Pad2)")
-	(net 114 "unconnected-(U34-NC_5-Pad5)")
-	(net 115 "unconnected-(U15-NC_26-Pad26)")
-	(net 116 "unconnected-(U15-NC_29-Pad29)")
-	(net 117 "unconnected-(U15-NC_30-Pad30)")
-	(net 118 "unconnected-(U15-NC_31-Pad31)")
-	(net 119 "unconnected-(U15-NC_32-Pad32)")
-	(net 120 "unconnected-(U15-NC_33-Pad33)")
-	(net 121 "unconnected-(U15-NC_34-Pad34)")
-	(net 122 "unconnected-(U15-NC_35-Pad35)")
-	(net 123 "unconnected-(U15-NC_38-Pad38)")
-	(net 124 "unconnected-(U15-NC_39-Pad39)")
-	(net 125 "unconnected-(U15-NC_42-Pad42)")
-	(net 126 "unconnected-(U15-NC_60-Pad60)")
-	(net 127 "unconnected-(U15-NC_61-Pad61)")
-	(net 128 "unconnected-(U17-NC_3-Pad3)")
-	(net 129 "unconnected-(U17-NC_12-Pad12)")
-	(net 130 "unconnected-(U17-NC_15-Pad15)")
-	(net 131 "unconnected-(U17-NC_29-Pad29)")
-	(net 132 "unconnected-(U17-NC_32-Pad32)")
-	(net 133 "unconnected-(U17-NC_33-Pad33)")
-	(net 134 "unconnected-(U17-NC_40-Pad40)")
-	(net 135 "unconnected-(J6-NC_A8-PadA8)")
-	(net 136 "unconnected-(J6-NC_B8-PadB8)")
 	(footprint "TestPoint:TestPoint_Pad_D1.0mm"
 		(layer "F.Cu")
@@
 			(layers "F.Cu" "F.Mask" "F.Paste")
 			(roundrect_rratio 0.05)
-			(net 105 "unconnected-(U16-NC_4-Pad4)")
 		)
 		(pad "5" smd roundrect
@@
 			(layers "F.Cu" "F.Mask" "F.Paste")
 			(roundrect_rratio 0.25)
-			(net 106 "unconnected-(U4-NC_2-Pad2)")
 		)
 		(pad "3" smd roundrect
@@
 			(layers "F.Cu" "F.Mask" "F.Paste")
 			(roundrect_rratio 0.25)
-			(net 107 "unconnected-(U4-NC_5-Pad5)")
 		)
 		(pad "6" smd roundrect
@@
 			(effects
 				(font
-					(size 0.8 0.8)
-					(thickness 0.15)
+					(size 0.7 0.7)
+					(thickness 0.12)
 				)
 			)
@@
 			(size 0.3 0.7)
 			(layers "F.Cu" "F.Mask" "F.Paste")
-			(net 108 "unconnected-(J21-NC_6-Pad6)")
 		)
 		(pad "MP" smd rect
@@
 			(size 0.3 1.3)
 			(layers "F.Cu" "F.Mask" "F.Paste")
-			(net 109 "unconnected-(J20-NC_13-Pad13)")
 		)
 		(pad "14" smd rect
@@
 			(size 0.5 0.2)
 			(layers "B.Cu" "B.Mask" "B.Paste")
-			(net 110 "unconnected-(U12-NC_3-Pad3)")
 		)
 		(pad "4" smd rect
@@
 			(layers "B.Cu" "B.Mask" "B.Paste")
 			(roundrect_rratio 0.25)
-			(net 111 "unconnected-(D10-NC_2-Pad2)")
 		)
 		(pad "3" smd roundrect
@@
 			(size 1.35 2)
 			(layers "B.Cu" "B.Mask" "B.Paste")
-			(net 112 "unconnected-(J1-NC_6-Pad6)")
 		)
 		(embedded_fonts no)
@@
 			(layers "B.Cu" "B.Mask" "B.Paste")
 			(roundrect_rratio 0.25)
-			(net 113 "unconnected-(U34-NC_2-Pad2)")
 		)
 		(pad "3" smd roundrect
@@
 			(layers "B.Cu" "B.Mask" "B.Paste")
 			(roundrect_rratio 0.25)
-			(net 114 "unconnected-(U34-NC_5-Pad5)")
 		)
 		(pad "6" smd roundrect
@@
 			(size 0.9 1.5)
 			(layers "B.Cu" "B.Mask" "B.Paste")
-			(net 115 "unconnected-(U15-NC_26-Pad26)")
 		)
 		(pad "27" smd rect
@@
 			(size 1.5 0.9)
 			(layers "B.Cu" "B.Mask" "B.Paste")
-			(net 116 "unconnected-(U15-NC_29-Pad29)")
 		)
 		(pad "30" smd rect
@@
 			(size 1.5 0.9)
 			(layers "B.Cu" "B.Mask" "B.Paste")
-			(net 117 "unconnected-(U15-NC_30-Pad30)")
 		)
 		(pad "31" smd rect
@@
 			(size 1.5 0.9)
 			(layers "B.Cu" "B.Mask" "B.Paste")
-			(net 118 "unconnected-(U15-NC_31-Pad31)")
 		)
 		(pad "32" smd rect
@@
 			(size 1.5 0.9)
 			(layers "B.Cu" "B.Mask" "B.Paste")
-			(net 119 "unconnected-(U15-NC_32-Pad32)")
 		)
 		(pad "33" smd rect
@@
 			(size 1.5 0.9)
 			(layers "B.Cu" "B.Mask" "B.Paste")
-			(net 120 "unconnected-(U15-NC_33-Pad33)")
 		)
 		(pad "34" smd rect
@@
 			(size 1.5 0.9)
 			(layers "B.Cu" "B.Mask" "B.Paste")
-			(net 121 "unconnected-(U15-NC_34-Pad34)")
 		)
 		(pad "35" smd rect
@@
 			(size 1.5 0.9)
 			(layers "B.Cu" "B.Mask" "B.Paste")
-			(net 122 "unconnected-(U15-NC_35-Pad35)")
 		)
 		(pad "36" smd rect
@@
 			(size 1.5 0.9)
 			(layers "B.Cu" "B.Mask" "B.Paste")
-			(net 123 "unconnected-(U15-NC_38-Pad38)")
 		)
 		(pad "39" smd rect
@@
 			(size 1.5 0.9)
 			(layers "B.Cu" "B.Mask" "B.Paste")
-			(net 124 "unconnected-(U15-NC_39-Pad39)")
 		)
 		(pad "40" smd rect
@@
 			(size 0.4 0.8)
 			(layers "B.Cu" "B.Mask" "B.Paste")
-			(net 125 "unconnected-(U15-NC_42-Pad42)")
 		)
 		(pad "43" smd rect
@@
 			(size 0.8 0.4)
 			(layers "B.Cu" "B.Mask" "B.Paste")
-			(net 126 "unconnected-(U15-NC_60-Pad60)")
 		)
 		(pad "61" smd rect
@@
 			(size 0.8 0.4)
 			(layers "B.Cu" "B.Mask" "B.Paste")
-			(net 127 "unconnected-(U15-NC_61-Pad61)")
 		)
 		(zone
@@
 			(layers "B.Cu" "B.Mask" "B.Paste")
 			(roundrect_rratio 0.25)
-			(net 128 "unconnected-(U17-NC_3-Pad3)")
 		)
 		(pad "4" smd roundrect
@@
 			(layers "B.Cu" "B.Mask" "B.Paste")
 			(roundrect_rratio 0.25)
-			(net 129 "unconnected-(U17-NC_12-Pad12)")
 		)
 		(pad "13" smd roundrect
@@
 			(layers "B.Cu" "B.Mask" "B.Paste")
 			(roundrect_rratio 0.25)
-			(net 130 "unconnected-(U17-NC_15-Pad15)")
 		)
 		(pad "16" smd roundrect
@@
 			(layers "B.Cu" "B.Mask" "B.Paste")
 			(roundrect_rratio 0.25)
-			(net 131 "unconnected-(U17-NC_29-Pad29)")
 		)
 		(pad "30" smd roundrect
@@
 			(layers "B.Cu" "B.Mask" "B.Paste")
 			(roundrect_rratio 0.25)
-			(net 132 "unconnected-(U17-NC_32-Pad32)")
 		)
 		(pad "33" smd roundrect
@@
 			(layers "B.Cu" "B.Mask" "B.Paste")
 			(roundrect_rratio 0.25)
-			(net 133 "unconnected-(U17-NC_33-Pad33)")
 		)
 		(pad "34" smd roundrect
@@
 			(layers "B.Cu" "B.Mask" "B.Paste")
 			(roundrect_rratio 0.25)
-			(net 134 "unconnected-(U17-NC_40-Pad40)")
 		)
 		(pad "41" smd rect
@@
 			(size 0.3 1.1)
 			(layers "B.Cu" "B.Mask" "B.Paste")
-			(net 135 "unconnected-(J6-NC_A8-PadA8)")
 		)
 		(pad "B1_A12" smd rect
@@
 			(size 0.3 1.1)
 			(layers "B.Cu" "B.Mask" "B.Paste")
-			(net 136 "unconnected-(J6-NC_B8-PadB8)")
 		)
 		(pad "S1" thru_hole oval
