File: hardware/pcb/hauptplatine/tools/routing/stand_vor_review_fixes.kicad_pcb (KiCad board)
At the start: 4 copper layers, 41 x 97 mm, 158 parts, among them J1 SJ-43504-SMT-TR, J20 503480-3000, J21 503480-0600, J4 microSD, J6 USB, Q1 PMV48XPA2R, Q10 2N7002T, Q11 2N7002T, Q20 2N7002T, Q21 2N7002T, Q22 2N7002T, SW1 B3U-3000P, SW2 B3U-3000P, SW3 B3U-3000P, U10 MCP73871, U12 TUSB320LAI, U15 ESP32-S31-WROOM-1-N16R16V, U16 TPS22948, U17 CS43131-CNZR, U20 TPS61023DRL, U21 TPS2553DRV, U22 MAX17048G+T10, U3 D5V0L2B3T-7, U30 PCA9306DCUR, U31 SN74AXC1T45DRL, U32 SN74AXC1T45DRL, U33 SN74AXC1T45DRL, U34 TLV75518PDRV, U4 TLV75733PDRV, U5 PE1605C4A6, X1 22.5792MHz, X2 24.576MHz

Commit message: Hauptplatine Rev. 3b: Review-Fixes (B1-B3, H1, H4, H5, H7, H8), Doku
Co-Authored-By: Claude Sonnet 5.5 <noreply@anthropic.com>
Claude-Session: https://claude.ai/code/session_01JifvE6gExGmwsJWDpfRrrS
Parts:
- removed Q21, Q22: 2N7002T, Package_TO_SOT_SMD:SOT-523
- removed R250: 100k, Resistor_SMD:R_0402_1005Metric
- removed SW2, SW3: B3U-3000P, Button_Switch_SMD:SW_SPST_B3U-3000P
- C257: value 100pF -> 100nF
- J20: value 503480-3000 -> FH12-30S-0.5SH(55); footprint Hauptplatine:Molex_503480-3000 -> Connector_FFC-FPC:Hirose_FH12-30S-0.5SH_1x30-1MP_P0.50mm_Horizontal
- R39: value 2.7k -> 1k
- moved J20 0.15 mm to (100.0, 100.5)
Connections:
- C257 pad 1: PCA_EN -> 3V3
- R36 pad 1: VBUS_SW -> 3V3
- R43 pad 1: GND -> 3V3
- U15 pad 48: unconnected-(U15-NC_48-Pad48) -> CHG_PROG2
- U15 pad 49: unconnected-(U15-NC_49-Pad49) -> CHG_SEL
- U30 pad 7: PCA_EN -> 3V3
Routing:
- net CHG_SEL: track 20.9 -> 79.6 mm, vias 1 -> 2
- net CHG_PROG2: track 14.2 -> 68.1 mm
- net ESP_EN: track 45.1 -> 7.22 mm, vias 7 -> 1
- net BOOT: track 43.9 -> 8.55 mm, vias 2 -> 1
- net SYS_POWER: track 147.9 -> 119.1 mm, vias 14 -> 7
- net GND: track 157.1 -> 128.7 mm
- net 3V3: track 294.5 -> 308.0 mm, vias 14 -> 11
- net DAC_RESET_N: track 25.6 -> 15.9 mm, vias 4 -> 2
- net VBUS_SW: track 20.2 -> 11.5 mm, vias 1 -> 0
- net RST_G: track 4.75 -> 0.00 mm
- net USB_DP: track 91.0 -> 86.5 mm, vias 3 -> 5
- net PCA_EN: track 14.0 -> 10.7 mm
- net USB_DN: track 90.5 -> 87.7 mm, vias 2 -> 3
- net VBUS: track 55.1 -> 57.2 mm, vias 9 -> 5
- net VBAT: track 116.5 -> 118.2 mm, vias 12 -> 5
