File: hardware/pcb/hauptplatine/hauptplatine.kicad_sch (KiCad schematic)
At the start: 71 parts, among them J1 AXE534124, J2 SM06B-SRSS-TB, J3 SM02B-SRSS-TB, J4 SJ-3524-SMT, J5 microSD, SW1 B3U-3000P, U1 XIAO ESP32S3 Plus, U2 TLV320DAC3100, U3 TPS7A2030PDBVR, U4 TLV75518PDBVR, U5 MAX17048G+T10

Commit message: Zwischenstand vor Pause: Klickrad v2 und Hauptplatine (unvollständig)
Beide Pakete wurden auf Wunsch angehalten. Klickrad v1 (MPR121) ist der
letzte fertige Stand der Klickrad-Platine in der Historie.

Co-Authored-By: Claude Opus 5.5 <noreply@anthropic.com>
Claude-Session: https://claude.ai/code/session_01JifvE6gExGmwsJWDpfRrrS
Parts:
- removed C11, C21, C28: 1uF, Capacitor_SMD:C_0402_1005Metric, symbol Device:C
- removed C20, C26: 4.7uF, Capacitor_SMD:C_0603_1608Metric, symbol Device:C
- removed C22: 100uF, Capacitor_SMD:C_0805_2012Metric, symbol Device:C
- removed C5: 100nF, Capacitor_SMD:C_0402_1005Metric, symbol Device:C
- removed C8: 22uF, Capacitor_SMD:C_0805_2012Metric, symbol Device:C
- removed J1: AXE534124, Tangara:FPC-AXE534124, symbol Tangara:FPC_34
- removed J2: SM06B-SRSS-TB, Connector_JST:JST_SH_SM06B-SRSS-TB_1x06-1MP_P1.00mm_Horizontal, symbol Connector_Generic:Conn_01x06
- removed J3: SM02B-SRSS-TB, Connector_JST:JST_SH_SM02B-SRSS-TB_1x02-1MP_P1.00mm_Horizontal, symbol Connector_Generic:Conn_01x02
- removed J4: SJ-3524-SMT, Connector_Audio:Jack_3.5mm_CUI_SJ-3524-SMT_Horizontal, symbol Tangara:Jack3_SwitchT
- removed J5: microSD, Connector_Card:microSD_HC_Molex_104031-0811, symbol Tangara:MicroSD
- removed R10: 4.7k, Resistor_SMD:R_0402_1005Metric, symbol Device:R
- removed R13, R14, R16, R17, R18, R19, R20, R21, R24: 10k, Resistor_SMD:R_0402_1005Metric, symbol Device:R
- removed R23: 100k, Resistor_SMD:R_0402_1005Metric, symbol Device:R
- removed TP1: TP_INT, TestPoint:TestPoint_Pad_D1.0mm, symbol Connector:TestPoint
- removed TP2: ALRT, TestPoint:TestPoint_Pad_D1.0mm, symbol Connector:TestPoint
- removed U1: XIAO ESP32S3 Plus, Tangara:XIAO-ESP32-S3-Plus-SMD, symbol Tangara:XIAO_ESP32S3_Plus
- removed U2: TLV320DAC3100, Package_DFN_QFN:Texas_RHB0032E_VQFN-32-1EP_5x5mm_P0.5mm_EP3.45x3.45mm, symbol Tangara:TLV320DAC3100
- removed U3: TPS7A2030PDBVR, Package_TO_SOT_SMD:SOT-23-5, symbol Tangara:LDO_SOT23_5
- removed U4: TLV75518PDBVR, Package_TO_SOT_SMD:SOT-23-5, symbol Tangara:LDO_SOT23_5
- removed U5: MAX17048G+T10, Package_DFN_QFN:TDFN-8-1EP_2x2mm_P0.5mm_EP0.8x1.2mm, symbol Tangara:MAX17048
- added C100: 1uF, Capacitor_SMD:C_0402_1005Metric, symbol Device:C
- added C101, C112: 22uF, Capacitor_SMD:C_0805_2012Metric, symbol Device:C
- added C102, C103, C104, C110, C114, C131, C133, C211: 100nF, Capacitor_SMD:C_0402_1005Metric, symbol Device:C
- added C111, C113, C130, C132, C32, C35, C42: 10uF, Capacitor_SMD:C_0805_2012Metric, symbol Device:C
- added C31, C34, C37, C39, C9: 0.1uF, Capacitor_SMD:C_0603_1608Metric, symbol Device:C
- added C38: 22uF, Capacitor_SMD:C_1206_3216Metric, symbol Device:C
- added D10: BAT54C, Package_TO_SOT_SMD:SOT-23, symbol Hauptplatine:D10
- added D4: BAT54C, Package_TO_SOT_SMD:SOT-23, symbol Hauptplatine:D4
- added J1: SJ-3506-SMT, Hauptplatine:CUI_SJ-3506-SMT, symbol Hauptplatine:J1
- added J20: AXE534124, Hauptplatine:FPC-AXE534124, symbol Hauptplatine:J20
- added J21: SM06B-SRSS-TB, Connector_JST:JST_SH_SM06B-SRSS-TB_1x06-1MP_P1.00mm_Horizontal, symbol Hauptplatine:J21
- added J4: microSD, Connector_Card:microSD_HC_Molex_104031-0811, symbol Hauptplatine:J4
- added J6: USB, Hauptplatine:GCT_USB4510-03-1-A_REVA, symbol Hauptplatine:J6
- added J7: Battery, Connector_JST:JST_SH_SM03B-SRSS-TB_1x03-1MP_P1.00mm_Horizontal, symbol Hauptplatine:J7
- added L1, L2: 4.7uH, Inductor_SMD:L_1008_2520Metric, symbol Device:L
- added L20: 1uH, Inductor_SMD:L_1008_2520Metric, symbol Device:L
- added Q1: PMV48XPA2R, Package_TO_SOT_SMD:TSOT-23, symbol Hauptplatine:Q_PMOS_123
- added Q10, Q11, Q3: PJC138K, Package_TO_SOT_SMD:SOT-323_SC-70, symbol Hauptplatine:Q_NMOS_123
- added R100, R101, R111, R115, R119, R122, R130, R131, R132, R133, R136, R137: 10k, Resistor_SMD:R_0402_1005Metric, symbol Device:R
- added R102, R103, R210, R211: 0, Resistor_SMD:R_0402_1005Metric, symbol Device:R
- added R110: 887k, Resistor_SMD:R_0402_1005Metric, symbol Device:R
- added R112, R113, R114, R135: 100k, Resistor_SMD:R_0402_1005Metric, symbol Device:R
- added R116: 390k, Resistor_SMD:R_0402_1005Metric, symbol Device:R
- added R117: 51k, Resistor_SMD:R_0402_1005Metric, symbol Device:R
- added R118: 49.9k, Resistor_SMD:R_0402_1005Metric, symbol Device:R
- added R120, R121: 2.2k, Resistor_SMD:R_0402_1005Metric, symbol Device:R
- added R134: 4.7k, Resistor_SMD:R_0402_1005Metric, symbol Device:R
- added R200, R202, R36: 100k, Resistor_SMD:R_0603_1608Metric, symbol Device:R
- added R201, R34, R35, R37, R38, R41, R43, R57, R61: 10k, Resistor_SMD:R_0603_1608Metric, symbol Device:R
- added R39: 1k, Resistor_SMD:R_0603_1608Metric, symbol Device:R
- added SW10: EN, Button_Switch_SMD:SW_SPST_B3U-1000P, symbol Switch:SW_Push
- added SW11: BOOT, Button_Switch_SMD:SW_SPST_B3U-1000P, symbol Switch:SW_Push
- added TP10: TX0, TestPoint:TestPoint_Pad_D1.0mm, symbol Connector:TestPoint
- added TP11: RX0, TestPoint:TestPoint_Pad_D1.0mm, symbol Connector:TestPoint
- added TP12: IO34 USB-JTAG D+, TestPoint:TestPoint_Pad_D1.0mm, symbol Connector:TestPoint
- added TP13: IO33 USB-JTAG D-, TestPoint:TestPoint_Pad_D1.0mm, symbol Connector:TestPoint
- added TP14: EN, TestPoint:TestPoint_Pad_D1.0mm, symbol Connector:TestPoint
- added TP15: BOOT, TestPoint:TestPoint_Pad_D1.0mm, symbol Connector:TestPoint
- added TP5: AMP_EN, TestPoint:TestPoint_Pad_D1.0mm, symbol Connector:TestPoint
- added TP6: AMP_MUTE, TestPoint:TestPoint_Pad_D1.0mm, symbol Connector:TestPoint
- added TP7: BAT, TestPoint:TestPoint_Pad_D1.0mm, symbol Connector:TestPoint
- added U1: INA1620, Package_DFN_QFN:Texas_RTW_WQFN-24-1EP_4x4mm_P0.5mm_EP2.7x2.7mm, symbol Hauptplatine:U1
- added U10: MCP73871, Package_DFN_QFN:QFN-20-1EP_4x4mm_P0.5mm_EP2.5x2.5mm, symbol Hauptplatine:U10
- added U12: TUSB320LAI, Hauptplatine:X2QFN-12-RWB, symbol Hauptplatine:U12
- added U15: ESP32-S31-WROOM-3-N16R16V, Hauptplatine:ESP32-S31-WROOM-3, symbol Hauptplatine:U15
- added U16: TPS22948, Hauptplatine:SOT65P210X110-6N, symbol Hauptplatine:U16
- added U17: WM8523, Package_SO:SSOP-20_4.4x6.5mm_P0.65mm, symbol Hauptplatine:U17
- added U20: TPS61023DRL, Package_TO_SOT_SMD:SOT-563, symbol Hauptplatine:U20
- added U21: TPS2553DBV, Package_TO_SOT_SMD:SOT-23-6, symbol Hauptplatine:U21
- added U22: MAX17048G+T10, Package_DFN_QFN:TDFN-8-1EP_2x2mm_P0.5mm_EP0.8x1.2mm, symbol Hauptplatine:U22
- added U3: D5V0L2B3T-7, Package_TO_SOT_SMD:SOT-523, symbol Hauptplatine:U3
- added U4: TLV75733PDBV, Package_TO_SOT_SMD:SOT-23-5, symbol Hauptplatine:U4
- added U5: PE1605C4A6, Package_TO_SOT_SMD:SOT-23-6, symbol Hauptplatine:U5
- added U7: TPS65133, Hauptplatine:SON40P300X300X80-13N, symbol Hauptplatine:U7
- added X1: Osc 22.5792MHz, Oscillator:Oscillator_SMD_Abracon_ASE-4Pin_3.2x2.5mm, symbol Hauptplatine:X1
- C1: value 100nF -> 10uF; footprint Capacitor_SMD:C_0402_1005Metric -> Capacitor_SMD:C_0805_2012Metric; Beschreibung Entprellung Ein/Aus 100 nF X7R 16 V -> (none); Herkunft (none) -> Tangara; Hersteller Samsung -> Murata; LCSC C1525 -> (none); MPN CL05B104KO5NNNC -> GRM21BR61C106KE15K; Tangara-Ref (none) -> C1
- C10: value 100nF -> 22uF; footprint Capacitor_SMD:C_0402_1005Metric -> Capacitor_SMD:C_1206_3216Metric; Beschreibung IOVDD 100 nF X7R 16 V -> (none); Herkunft (none) -> Tangara; Hersteller Samsung -> Murata; LCSC C1525 -> (none); MPN CL05B104KO5NNNC -> GRM319R61C226KE15D; Tangara-Ref (none) -> C10
- C12: value 100nF -> 1uF; footprint Capacitor_SMD:C_0402_1005Metric -> Capacitor_SMD:C_0805_2012Metric; Beschreibung DVDD 100 nF X7R 16 V -> (none); Herkunft (none) -> Tangara; Hersteller Samsung -> Murata; LCSC C1525 -> (none); MPN CL05B104KO5NNNC -> GRM216R61C105KA88D; Tangara-Ref (none) -> C12
- C13: value 4.7uF -> 0.1uF; Beschreibung DVDD 4,7 uF X5R 16 V -> (none); Herkunft (none) -> Tangara; Hersteller Samsung -> Murata; MPN CL10A475KO8NNNC -> GCM188R71C104KA37J; Tangara-Ref (none) -> C13
- C14: value 100nF -> 0.1uF; footprint Capacitor_SMD:C_0402_1005Metric -> Capacitor_SMD:C_0603_1608Metric; Beschreibung AVDD 100 nF X7R 16 V -> (none); Herkunft (none) -> Tangara; Hersteller Samsung -> Murata; LCSC C1525 -> (none); MPN CL05B104KO5NNNC -> GCM188R71C104KA37J; Tangara-Ref (none) -> C14
- C15: value 4.7uF -> 2700pF; Beschreibung AVDD 4,7 uF X5R 16 V -> (none); Herkunft (none) -> Tangara; Hersteller Samsung -> Murata; MPN CL10A475KO8NNNC -> GRM1885C1H272JA01J; Tangara-Ref (none) -> C15
- C16: value 100nF -> 22uF; footprint Capacitor_SMD:C_0402_1005Metric -> Capacitor_SMD:C_1206_3216Metric; Beschreibung HPVDD 100 nF X7R 16 V -> (none); Herkunft (none) -> Tangara; Hersteller Samsung -> Murata; LCSC C1525 -> (none); MPN CL05B104KO5NNNC -> GRM319R61C226KE15D; Tangara-Ref (none) -> C16
- C17: value 4.7uF -> 100pF; Beschreibung HPVDD 4,7 uF X5R 16 V -> (none); Herkunft (none) -> Tangara; Hersteller Samsung -> (none); MPN CL10A475KO8NNNC -> (none); Tangara-Ref (none) -> C17
- C18: value 100nF -> 10uF; footprint Capacitor_SMD:C_0402_1005Metric -> Capacitor_SMD:C_0805_2012Metric; Beschreibung SPKVDD (Verstaerker unbenutzt) 100 nF X7R 16 V -> (none); Herkunft (none) -> Tangara; Hersteller Samsung -> Murata; LCSC C1525 -> (none); MPN CL05B104KO5NNNC -> GRM21BR61C106KE15K; Tangara-Ref (none) -> C18
- C19: value 100nF -> 100pF; footprint Capacitor_SMD:C_0402_1005Metric -> Capacitor_SMD:C_0603_1608Metric; Beschreibung SPKVDD 100 nF X7R 16 V -> (none); Herkunft (none) -> Tangara; Hersteller Samsung -> (none); LCSC C1525 -> (none); MPN CL05B104KO5NNNC -> (none); Tangara-Ref (none) -> C19
- C2: footprint Capacitor_SMD:C_0603_1608Metric -> Capacitor_SMD:C_0805_2012Metric; Beschreibung Display VCI/VDDIO 10 uF X5R 10 V -> (none); Herkunft (none) -> Tangara; Hersteller Samsung -> Murata; LCSC C19702 -> (none); MPN CL10A106KP8NNNC -> GRM21BR61C106KE15K; Tangara-Ref (none) -> C2
- C23: value 100uF -> 1uF; Beschreibung DC-Sperre Kopfhoerer rechts 100 uF X5R 6,3 V -> (none); Herkunft (none) -> Tangara; Hersteller Samsung -> Murata; MPN CL21A107MQYNNNE -> GRM216R61C105KA88D; Tangara-Ref (none) -> C23
- C24: value 1uF -> 10uF; footprint Capacitor_SMD:C_0402_1005Metric -> Capacitor_SMD:C_0805_2012Metric; Beschreibung U3 Eingang 1 uF X5R 6,3 V -> (none); Herkunft (none) -> Tangara; Hersteller Samsung -> Murata; LCSC C52923 -> (none); MPN CL05A105KA5NQNC -> GRM21BR61C106KE15K; Tangara-Ref (none) -> C24
- C25: value 1uF -> 10uF; footprint Capacitor_SMD:C_0402_1005Metric -> Capacitor_SMD:C_0805_2012Metric; Beschreibung U3 Ausgang 1 uF X5R 6,3 V -> (none); Herkunft (none) -> Tangara; Hersteller Samsung -> Murata; LCSC C52923 -> (none); MPN CL05A105KA5NQNC -> GRM21BR61C106KE15K; Tangara-Ref (none) -> C25
- C27: value 1uF -> 10uF; footprint Capacitor_SMD:C_0402_1005Metric -> Capacitor_SMD:C_0805_2012Metric; Beschreibung U4 Eingang 1 uF X5R 6,3 V -> (none); Herkunft (none) -> Tangara; Hersteller Samsung -> Murata; LCSC C52923 -> (none); MPN CL05A105KA5NQNC -> GRM21BR61C106KE15K; Tangara-Ref (none) -> C27
- C29: value 4.7uF -> 100uF; footprint Capacitor_SMD:C_0603_1608Metric -> Capacitor_SMD:C_1210_3225Metric; Beschreibung U4 Ausgang 4,7 uF X5R 16 V -> (none); Herkunft (none) -> Tangara; Hersteller Samsung -> Murata; MPN CL10A475KO8NNNC -> GRM32EC70J107ME15K; Tangara-Ref (none) -> C29
- C3: value 100nF -> 10uF; footprint Capacitor_SMD:C_0402_1005Metric -> Capacitor_SMD:C_0805_2012Metric; Beschreibung Display VCI/VDDIO 100 nF X7R 16 V -> (none); Herkunft (none) -> Tangara; Hersteller Samsung -> Murata; LCSC C1525 -> (none); MPN CL05B104KO5NNNC -> GRM21BR61C106KE15K; Tangara-Ref (none) -> C3
- C30: value 100nF -> 0.1uF; footprint Capacitor_SMD:C_0402_1005Metric -> Capacitor_SMD:C_0603_1608Metric; Beschreibung MAX17048 VDD 100 nF X7R 16 V -> (none); Herkunft (none) -> Tangara; Hersteller Samsung -> Murata; LCSC C1525 -> (none); MPN CL05B104KO5NNNC -> GCM188R71C104KA37J; Tangara-Ref (none) -> C30
- C4: value 10uF -> 1uF; footprint Capacitor_SMD:C_0603_1608Metric -> Capacitor_SMD:C_0805_2012Metric; Beschreibung Display/Touch VDD 10 uF X5R 10 V -> (none); Herkunft (none) -> Tangara; Hersteller Samsung -> Murata; LCSC C19702 -> (none); MPN CL10A106KP8NNNC -> GRM216R61C105KA88D; Tangara-Ref (none) -> C4
- C6: value 10uF -> 2700pF; Beschreibung SD VDD 10 uF X5R 10 V -> (none); Herkunft (none) -> Tangara; Hersteller Samsung -> Murata; LCSC C19702 -> (none); MPN CL10A106KP8NNNC -> GRM1885C1H272JA01J; Tangara-Ref (none) -> C6
- C7: value 100nF -> 10uF; footprint Capacitor_SMD:C_0402_1005Metric -> Capacitor_SMD:C_0805_2012Metric; Beschreibung SD VDD 100 nF X7R 16 V -> (none); Herkunft (none) -> Tangara; Hersteller Samsung -> Murata; LCSC C1525 -> (none); MPN CL05B104KO5NNNC -> GRM21BR61C106KE15K; Tangara-Ref (none) -> C7
- H1, H2, H3: Beschreibung Montageloch Abstandshalter Klickrad (Detail: README) -> Montageloch Abstandshalter Klickrad (NPTH 2,2 mm, r = 14,6 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; Herkunft (none) -> neu
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Connections:
- net HPR is gone; now on net 3V3: C23.1
- net HPR_J is gone; now on net GND: C23.2
- net 3V3: now also C1.1, C2.2, C29.1, C30.1, R2.2, R22.2, C101.1, C102.1, C110.1, C130.1, C131.1, C132.1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; no longer C10.1, C18.1, C19.1, C2.1, C24.1, C27.1, C4.1, C6.1, C7.1, R1.1, R11.1, R15.1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
- net FG_ALRT: now also R122.2, U15.21 (IO15), U22.5 (ALRT)
- net GND: now also C10.1, C12.1, C14.2, C15.1, C16.2, C18.2, C2.1, C24.2, C25.2, C6.1, R1.2, R3.1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; no longer C10.2, C12.2, C2.2, C4.2, C6.2, R22.2, R7.2, SW1.2
- net LCD_CS: now also J20.11 (CS), U15.63 (IO53)
- net LCD_D0: now also J20.5 (SIO0), U15.60 (IO50)
- net LCD_D1: now also J20.7 (SIO1), U15.61 (IO51)
- net LCD_D2: now also J20.13 (SIO2), U15.64 (IO54)
- net LCD_D3: now also J20.15 (SIO3), U15.65 (IO55)
- net LCD_IM0: now also J20.19 (IM0), R131.1; no longer R7.1
- net LCD_IM1: now also J20.17 (IM1), R130.2; no longer R6.2
- net LCD_PWR_EN: now also J20.22 (PWR_EN), R134.2
- net LCD_RST: now also J20.1 (RESET), R135.2, U15.55 (IO45); no longer R11.2
- net LCD_SCK: now also J20.9 (QSPI_SCL), U15.62 (IO52)
- net LCD_TE: now also J20.2 (TE), U15.59 (IO49); no longer R12.2
- net SCL: now also J20.8 (TP_SCL), J21.4 (SCL), R121.2, U12.8 (SCL/OUT2), U15.24 (IO18), U17.14 (SCLK), U22.7 (SCL); no longer R2.2
- net SDA: now also J20.10 (TP_SDA), J21.3 (SDA), R120.2, U12.7 (SDA/OUT1), U15.25 (IO19), U17.13 (SDA), U22.8 (SDA); no longer R1.2
- net SD_CLK: now also J4.5 (CLK), U15.31 (SD_CLK)
- net SD_CMD: now also R11.2, J4.3 (CMD), U15.32 (SD_CMD)
- net SD_D0: now also R9.2, J4.7 (DAT0), U15.27 (SD_D0)
- net SD_D1: now also J4.8 (DAT1), R57.2, U15.28 (SD_D1); no longer R15.2
- net SD_D2: now also J4.1 (DAT2), R61.2, U15.29 (SD_D2)
- net SD_D3: now also R12.2, J4.2 (DAT3), U15.30 (SD_D3)
- net TP_INT: now also J20.12 (TP_INT), R133.2, U15.54 (IO44); no longer R9.2
- net TP_RST: now also J20.14 (TP_RST), R132.2; no longer R8.2
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Other:
- note added: "AMOLED-Anschluss (FPC 34 Pol, wie Waveshare ESP32-S3-Touch-AMOLED-1.8)"
- note added: "Audio: WM8523 + INA1620 + TPS65133 + Klinke (1:1 von Tangara, + MCLK-Option)"
- note added: "ESP32-S31-WROOM-3 (Espressif-Beschaltung)"
- note added: "Klickrad-Anschluss (JST-SH 6 Pol), Montagelocher"
- note added: "PWR_FLAGs fuer ERC (Speisenetze werden von Bauteilen mit passiven Pins gespeist)"
- note added: "Power: MCP73871 + TLV75733 + Akku + Power-Latch (von Tangara, angepasst), Fuel Gauge MAX17048"
- note added: "USB-C Dual-Role + Host-VBUS (TUSB320 + TPS61023 + TPS2553): EIGENE ENTWICKLUNG, UNGEPRUEFT; ESD wie Tangara"
- note added: "microSD (SDMMC 4 Bit) + Lastschalter TPS22948"
- note removed: "Audio: TLV320DAC3100, I2S + I2C 0x18, PLL aus BCLK (MCLK auf GND), AVDD 3,0 V / DVDD 1,8 V eigene LDOs"
- note removed: "Display-Anschluss (34 Pin, Belegung wie Waveshare ESP32-S3-Touch-AMOLED-1.8, CO5300 QSPI 368x448)"
- note removed: "Display-Entkopplung, Reset, IM-Pins, Touch"
- note removed: "Ein/Aus-Taster: seitlich betaetigter Taster an der Oberkante (Oberseite)"
- note removed: "Fuel Gauge MAX17048 (I2C 0x36), Akkuanschluss"
- note removed: "I2C-Pull-ups (Bus: DAC 0x18, MAX17048 0x36, Klickrad 0x5A/0x5B, Touch 0x15/0x38), Klickrad-Pull-ups, Ein/Aus-Taster"
- note removed: "Klickrad-Modul (SM06B-SRSS-TB, Belegung laut TEILE.md)"
- note removed: "Klinkenbuchse mit Steckererkennung (Schliesser TN an der Spitze)"
- note removed: "Montagelocher Klickrad (NPTH 2,2 mm, r = 14,6 mm um (0,-27) bei 90/210/330 Grad)"
- note removed: "Spannungsversorgung Audio: U3 AVDD 3,0 V (analog, auf AGND), U4 DVDD 1,8 V"
- note removed: "XIAO ESP32S3 Plus (SMD-Montage): GPIO-Zuordnung siehe README / Pin-Tabelle"
- note removed: "microSD (SDMMC 1-Bit), Pull-ups"
- title: Hauptplatine Nano-Player (Endgeraet) -> Hauptplatine Nano-Player (Endgeraet), Rev. 1

Commit message: Platinen: Zwischenstand (in Arbeit)
Co-Authored-By: Claude Opus 5.5 <noreply@anthropic.com>
Claude-Session: https://claude.ai/code/session_01JifvE6gExGmwsJWDpfRrrS
Parts:
- removed C1, C18, C2, C3, C7: 10uF, Capacitor_SMD:C_0805_2012Metric, symbol Device:C
- removed C10, C16, C38: 22uF, Capacitor_SMD:C_1206_3216Metric, symbol Device:C
- removed C12, C4: 1uF, Capacitor_SMD:C_0805_2012Metric, symbol Device:C
- removed C13, C14, C31, C39, C9: 0.1uF, Capacitor_SMD:C_0603_1608Metric, symbol Device:C
- removed C15, C6: 2700pF, Capacitor_SMD:C_0603_1608Metric, symbol Device:C
- removed C17, C19: 100pF, Capacitor_SMD:C_0603_1608Metric, symbol Device:C
- removed C211: 100nF, Capacitor_SMD:C_0402_1005Metric, symbol Device:C
- removed J7: Battery, Connector_JST:JST_SH_SM03B-SRSS-TB_1x03-1MP_P1.00mm_Horizontal, symbol Hauptplatine:J7
- removed L1, L2: 4.7uH, Inductor_SMD:L_1008_2520Metric, symbol Device:L
- removed Q3: PJC138K, Package_TO_SOT_SMD:SOT-323_SC-70, symbol Hauptplatine:Q_NMOS_123
- removed R133, R137: 10k, Resistor_SMD:R_0402_1005Metric, symbol Device:R
- removed R15, R6: 560, Resistor_SMD:R_0805_2012Metric, symbol Device:R
- removed R2, R22, R5: 10k, Resistor_SMD:R_0603_1608Metric, symbol Device:R
- removed R210, R211: 0, Resistor_SMD:R_0402_1005Metric, symbol Device:R
- removed R3, R8: 2.2k, Resistor_SMD:R_0805_2012Metric, symbol Device:R
- removed SW10: EN, Button_Switch_SMD:SW_SPST_B3U-1000P, symbol Switch:SW_Push
- removed SW11: BOOT, Button_Switch_SMD:SW_SPST_B3U-1000P, symbol Switch:SW_Push
- removed TP3: +5V, TestPoint:TestPoint_Pad_D1.0mm, symbol Connector:TestPoint
- removed TP4: -5V, TestPoint:TestPoint_Pad_D1.0mm, symbol Connector:TestPoint
- removed TP5: AMP_EN, TestPoint:TestPoint_Pad_D1.0mm, symbol Connector:TestPoint
- removed TP6: AMP_MUTE, TestPoint:TestPoint_Pad_D1.0mm, symbol Connector:TestPoint
- removed U1: INA1620, Package_DFN_QFN:Texas_RTW_WQFN-24-1EP_4x4mm_P0.5mm_EP2.7x2.7mm, symbol Hauptplatine:U1
- removed U7: TPS65133, Hauptplatine:SON40P300X300X80-13N, symbol Hauptplatine:U7
- added BT1: Akku 3-pol., Hauptplatine:BATT_PADS_3, symbol Hauptplatine:BT1
- added C240, C241, C242, C253, C257, C258, C259, C262: 100nF, Capacitor_SMD:C_0402_1005Metric, symbol Device:C
- added C243, C244, C247, C248, C249, C250, C251, C252, C261: 2.2uF, Capacitor_SMD:C_0402_1005Metric, symbol Device:C
- added C245, C246: 15uF, Capacitor_SMD:C_0603_1608Metric, symbol Device:C
- added C254: 4.7uF, Capacitor_SMD:C_0603_1608Metric, symbol Device:C
- added C255, C256: 10pF, Capacitor_SMD:C_0402_1005Metric, symbol Device:C
- added C260: 1uF, Capacitor_SMD:C_0402_1005Metric, symbol Device:C
- added FB1: BLM15 120R, Inductor_SMD:L_0402_1005Metric, symbol Device:L
- added H4: M1.6, Hauptplatine:MountingHole_1.8mm, symbol Mechanical:MountingHole
- added Q20: 2N7002T, Package_TO_SOT_SMD:SOT-523, symbol Hauptplatine:Q_NMOS_123
- added R240, R241, R242, R243: 0, Resistor_SMD:R_0402_1005Metric, symbol Device:R
- added R244, R245: 100k, Resistor_SMD:R_0402_1005Metric, symbol Device:R
- added R246: 10k, Resistor_SMD:R_0402_1005Metric, symbol Device:R
- added R247: 200k, Resistor_SMD:R_0402_1005Metric, symbol Device:R
- added R248, R249: 4.7k, Resistor_SMD:R_0402_1005Metric, symbol Device:R
- added TP16: GND neben EN, TestPoint:TestPoint_Pad_D1.0mm, symbol Connector:TestPoint
- added TP17: GND neben BOOT, TestPoint:TestPoint_Pad_D1.0mm, symbol Connector:TestPoint
- added U30: PCA9306DCUR, Package_SO:VSSOP-8_2.3x2mm_P0.5mm, symbol Hauptplatine:U30
- added U31: SN74AXC1T45DRL, Package_TO_SOT_SMD:SOT-563, symbol Hauptplatine:U31
- added U32: SN74AXC1T45DRL, Package_TO_SOT_SMD:SOT-563, symbol Hauptplatine:U32
- added U33: SN74AXC1T45DRL, Package_TO_SOT_SMD:SOT-563, symbol Hauptplatine:U33
- added U34: TLV75518PDRV, Package_SON:WSON-6-1EP_2x2mm_P0.65mm_EP1x1.6mm, symbol Hauptplatine:U34
- added X2: 24.576MHz, Crystal:Crystal_SMD_2016-4Pin_2.0x1.6mm, symbol Hauptplatine:X2
- C101, C112: footprint Capacitor_SMD:C_0805_2012Metric -> Capacitor_SMD:C_0603_1608Metric; Hersteller Samsung -> Murata; LCSC C45783 -> (none); MPN CL21A226MAQNNNE -> GRM188R60J226MEA0
- C103: Beschreibung Entprellung Boot-Taster -> Entprellung/Filter BOOT
- C111, C113: footprint Capacitor_SMD:C_0805_2012Metric -> Capacitor_SMD:C_0603_1608Metric; MPN GRM21BR61C106KE15K -> GRM188R61A106KE69
- C130: footprint Capacitor_SMD:C_0805_2012Metric -> Capacitor_SMD:C_0402_1005Metric; Beschreibung Display-Versorgung (Waveshare C24/C25/C27/C28) -> Display-Versorgung VCI/VDDIO (Waveshare C27); MPN GRM21BR61C106KE15K -> GRM155R60J106ME05D
- C131: Beschreibung Display-Versorgung (Waveshare C24/C25/C27/C28) -> Display-Versorgung VCI/VDDIO (Waveshare C28)
- C132: footprint Capacitor_SMD:C_0805_2012Metric -> Capacitor_SMD:C_0402_1005Metric; Beschreibung Display-Versorgung (Waveshare C24/C25/C27/C28) -> Touch-Versorgung (Waveshare C25); MPN GRM21BR61C106KE15K -> GRM155R60J106ME05D
- C133: Beschreibung Display-Versorgung (Waveshare C24/C25/C27/C28) -> Touch-Versorgung (Waveshare C24)
- C23: footprint Capacitor_SMD:C_0805_2012Metric -> Capacitor_SMD:C_0603_1608Metric; Beschreibung (none) -> 0603 statt 0805 (Hoehe <= 1,0 mm fuer die Oberseite); Herkunft Tangara -> angepasst; MPN GRM216R61C105KA88D -> GRM188R61A105KA61D
- C24, C25, C27, C32, C35, C42: footprint Capacitor_SMD:C_0805_2012Metric -> Capacitor_SMD:C_0603_1608Metric; Beschreibung (none) -> 0603 statt 0805 (Hoehe <= 1,0 mm fuer die Oberseite); Herkunft Tangara -> angepasst; MPN GRM21BR61C106KE15K -> GRM188R61A106KE69
- H1, H2, H3: value M2-Klickrad -> M1.6; footprint MountingHole:MountingHole_2.2mm_M2 -> Hauptplatine:MountingHole_1.8mm; Beschreibung Montageloch Abstandshalter Klickrad (NPTH 2,2 mm, r = 14,6 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 -> Gehaeuse-Befestigung M1,6 (NPTH 1,8 mm), Position zur Absti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
- J1: value SJ-3506-SMT -> SJ-43504-SMT-TR; footprint Hauptplatine:CUI_SJ-3506-SMT -> Hauptplatine:CUI_SJ-43504-SMT-TR; Beschreibung (none) -> Klinke 5,0 mm hoch (Tangara: SJ-3506-SMT, 6,0 mm), Mid-Moun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; Herkunft Tangara -> angepasst; Hersteller CUI Devices -> Same Sky (CUI Devices); MPN SJ-3506-SMT-TR -> SJ-43504-SMT-TR; Tangara-Ref J1 -> (none)
- J20: value AXE534124 -> FH12-30S-0.5SH(55); footprint Hauptplatine:FPC-AXE534124 -> Connector_FFC-FPC:Hirose_FH12-30S-0.5SH_1x30-1MP_P0.50mm_Horizontal; Beschreibung Display-FPC-Buchse wie Waveshare ESP32-S3-Touch-AMOLED-1.8 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 -> Display-FPC-Stecker, 30 Pin 0,5 mm (Waveshare 2,06'-Board J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; Hersteller Panasonic -> Hirose; MPN AXE534124 -> FH12-30S-0.5SH(55)
- J21: value SM06B-SRSS-TB -> FH12-6S-0.5SH(55); footprint Connector_JST:JST_SH_SM06B-SRSS-TB_1x06-1MP_P1.00mm_Horizontal -> Connector_FFC-FPC:Hirose_FH12-6S-0.5SH_1x06-1MP_P0.50mm_Horizontal; Beschreibung Klickrad-Modul (Belegung laut TEILE.md; Pin 5 = INT/CHANGE,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 -> Klickrad-Modul v2 (AT42QT2120 0x1C + DRV2605L 0x5A), gleich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; DigiKey 455-SM06B-SRSS-TBCT-ND -> (none); Hersteller JST -> Hirose; LCSC C160405 -> (none); MPN SM06B-SRSS-TB(LF)(SN) -> FH12-6S-0.5SH(55)
- J4: Beschreibung microSD statt Vollformat-SD (Tangara: Hirose DM1AA-SF-PEJ(82), 32 x 32 mm); SDMMC 4 Bit direkt am S31 statt SPI + Multiplexer -> microSD statt Vollformat-SD (Tangara: Hirose DM1AA-SF-PEJ(82)); SDMMC 4 Bit direkt am S31 (IO35...IO40) statt SPI + Multiplexer
- L20: footprint Inductor_SMD:L_1008_2520Metric -> Inductor_SMD:L_0805_2012Metric; Beschreibung 1 uH (TPS61023 Tab. 8-2), Saettigungsstrom >= 3 A; Typ vor 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 -> 1 uH 2,0 x 1,6 x 1,0 mm (TPS61023 Tab. 8-2: Saettigungsstro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; MPN DFE252012F-1R0M=P2 -> DFE201610E-1R0M=P2
- Q10, Q11: value PJC138K -> 2N7002T; footprint Package_TO_SOT_SMD:SOT-323_SC-70 -> Package_TO_SOT_SMD:SOT-523; Hersteller PANJIT -> Diodes Inc.; MPN PJC138K_R1_00001 -> 2N7002T-7-F
- R102: Beschreibung USB-HS D+: Platz fuer Serienwiderstand (Espressif: nahe am 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 -> USB-HS D+: Platz fuer Serienwiderstand (Anfangswert 0 Ohm)
- R132: Beschreibung Touch-Reset hoch (immer aus dem Reset) -> Touch-Reset hoch (immer aus dem Reset; Waveshare: GPIO9)
- R134: Beschreibung FPC-Pin 22 (Waveshare DSI_PWR_EN) fest high -> FPC-Pin 21 (Waveshare DSI_PWR_EN) fest high
- R136: Beschreibung Pull-up Klickrad INT/CHANGE (open drain, aktiv low) -> Pull-up CHANGE (open drain, aktiv low)
- R36: Beschreibung PROG2 hoch = USB-Eingangslimit 500 mA (Tangara: Pin vom SAMD21 gesteuert); hier Pull-up an 3V3 (S31-GPIO darf nicht auf 5 V haengen), S31 kann ueberschreiben -> PROG2 hoch = USB-Eingangslimit 500 mA (Tangara: Pin vom SAMD21 gesteuert); hier Pull-up an 3V3, S31 kann ueberschreiben
- TP14: value EN -> EN (gegen TP16 kurzschliessen = Reset)
- TP15: value BOOT -> BOOT (gegen TP17 kurzschliessen = Download-Modus)
- U15: value ESP32-S31-WROOM-3-N16R16V -> ESP32-S31-WROOM-1-N16R16V; footprint Hauptplatine:ESP32-S31-WROOM-3 -> Hauptplatine:ESP32-S31-WROOM-1; Beschreibung WLAN 6, Bluetooth 5.4 (Classic + LE Audio), USB 2.0 HS OTG, 16 MB Flash (Quad), 16 MB PSRAM (Octal) (Datenblatt v0.7 PRELIMINARY); Tangara: ESP32-WROVER-E mit 8 MB PSRAM -> WLAN 6, Bluetooth 5.4 (Classic + LE Audio), USB 2.0 HS OTG, 16 MB Flash, 16 MB PSRAM (Datenblatt v0.5 PRELIMINARY); Tangara: ESP32-WROVER-E; MPN ESP32-S31-WROOM-3-N16R16V -> ESP32-S31-WROOM-1-N16R16V
- U17: value WM8523 -> CS43131-CNZR; footprint Package_SO:SSOP-20_4.4x6.5mm_P0.65mm -> Package_DFN_QFN:QFN-40-1EP_5x5mm_P0.4mm_EP3.6x3.6mm; Beschreibung (none) -> DAC mit Class-H-Kopfhoererverstaerker (125 dB DNR an 32 Ohm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; DigiKey (none) -> 598-CS43131-CNZRCT-ND; Herkunft Tangara -> neu; MPN WM8523GEDT/R -> CS43131-CNZR; Tangara-Ref U17 -> (none)
- U21: value TPS2553DBV -> TPS2553DRV; footprint Package_TO_SOT_SMD:SOT-23-6 -> Package_SON:WSON-6-1EP_2x2mm_P0.65mm_EP1x1.6mm; Beschreibung Lastschalter mit Strombegrenzung (49,9 k = ca. 520 mA) -> Lastschalter mit Strombegrenzung (49,9 k = ca. 520 mA), WSO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; DigiKey 296-32464-1-ND -> (none); LCSC C55266 -> (none); MPN TPS2553DBVR -> TPS2553DRVR
- U3: Beschreibung (none) -> ESD-Schutz Kopfhoerer-Ausgaenge (Tangara 1:1, Netze angepas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
- U4: value TLV75733PDBV -> TLV75733PDRV; footprint Package_TO_SOT_SMD:SOT-23-5 -> Package_SON:WSON-6-1EP_2x2mm_P0.65mm_EP1x1.6mm; Beschreibung 3V3-LDO 1 A statt 500 mA (TLV75533) -> 3V3-LDO 1 A (Tangara: TLV75533PDBV, 500 mA) im flachen WSON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; DigiKey 296-50414-1-ND -> (none); LCSC C485517 -> (none); MPN TLV75733PDBVR -> TLV75733PDRVR
- X1: value Osc 22.5792MHz -> 22.5792MHz; footprint Oscillator:Oscillator_SMD_Abracon_ASE-4Pin_3.2x2.5mm -> Crystal:Crystal_SMD_2016-4Pin_2.0x1.6mm; Beschreibung Optionaler MCLK-Oszillator, 3V3, nicht bestueckt (DNP) -> Quarz 22,5792 MHz, Last 8 pF, laut CS43131 Tab. 5-1 geeigne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; Herkunft neu -> Cirrus; Hersteller (none) -> NDK; MPN (Typ nach Abtastraten-Familie waehlen, z. B. 22,5792 MHz) -> NX2016SA 22.5792M EXS00A-CS09116; now fitted
Connections:
- net AMP_EN is gone; now on net USBJ_DP: U15.14 (IO34)
- net DAC_MCK_MCU is gone; now on an unnamed net: U15.15 (NC)
- net Q3_G is gone; now on an unnamed net: U15.17 (NC)
- net 3V3: now also J20.11 (TP_VDD), J20.23 (VCI), J20.25 (VDDIO), J20.29 (3V3), J20.30 (3V3), U15.2 (3V3), U4.1 (OUT), C257.1, C258.1, C259.1, C260.1, R244.1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; no longer J20.16 (TP_VDD), J20.18, J20.20, J20.24 (VCI), J20.26 (VDDIO), U15.3 (3V3), U15.4 (3V3), U17.19 (AVDD), U17.6 (LINEVDD), U4.5 (OUT), X1.1 (EN), X1.4 (VDD)
- net BOOT: now also U15.27 (IO61); no longer U15.71 (IO61)
- net CHG_PG: no longer U15.52 (IO42)
- net CHG_PROG2: no longer U15.49 (IO38)
- net CHG_SEL: no longer U15.50 (IO39)
- net CHG_STAT1: no longer U15.53 (IO43)
- net CHG_STAT2: no longer U15.51 (IO40)
- net ESP_EN: now also U15.3 (EN); no longer U15.5 (EN)
- net FG_ALRT: no longer U15.21 (IO15)
- net GND: now also J20.1 (GND), J20.16 (GND), J20.18 (GND), J20.2 (GND), J20.20 (GND), J20.22 (GND), J20.24 (GND), J20.26 (GND), J20.MP (GND), U15.40 (GND), U15.41 (GND), U17.19 (GND)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; no longer J1.1 (GND), J1.5 (GND), J1.SH1 (GND), J1.SH2 (GND), J20.21 (GND), J20.23 (GND), J20.25 (GND), J20.27 (GND), J20.29 (GND), J20.3 (GND), J20.31 (GND), J20.33 (GND)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
- net HOST_EN: now also U21.4 (EN); no longer U15.23 (IO17), U21.3 (EN)
- net HOST_FLT: now also U21.3 (FAULT); no longer U21.4 (FAULT)
- net HOST_ILIM: now also U21.2 (ILIM); no longer U21.5 (ILIM)
- net KEY_LOCK_MCU: no longer U15.6 (IO2)
- net LCD_CS: now also J20.6 (LCD_CS); no longer J20.11 (CS), U15.63 (IO53)
- net LCD_D0: now also J20.14 (QSPI_SIO0); no longer J20.5 (SIO0), U15.60 (IO50)
- net LCD_D1: now also J20.12 (QSPI_SIO1); no longer J20.7 (SIO1), U15.61 (IO51)
- net LCD_D2: now also J20.10 (QSPI_SIO2); no longer J20.13 (SIO2), U15.64 (IO54)
- net LCD_D3: now also J20.8 (QSPI_SIO3); no longer J20.15 (SIO3), U15.65 (IO55)
- net LCD_IM0: now also J20.17 (IM0); no longer J20.19 (IM0)
- net LCD_IM1: now also J20.15 (IM1); no longer J20.17 (IM1)
- net LCD_PWR_EN: now also J20.21 (DSI_PWR_EN); no longer J20.22 (PWR_EN)
- net LCD_RST: now also J20.19 (LCD_RESET); no longer J20.1 (RESET), U15.55 (IO45)
- net LCD_SCK: now also J20.4 (QSPI_SCL); no longer J20.9 (QSPI_SCL), U15.62 (IO52)
- net LCD_TE: now also J20.27 (LCD_TE); no longer J20.2 (TE), U15.59 (IO49)
- net LDO_EN: now also U4.4 (EN); no longer U4.3 (EN)
- net NTC: now also BT1.1 (NTC)
- net SCL: now also J20.3 (TP_SCL), U30.6 (SCL2); no longer J20.8 (TP_SCL), U15.24 (IO18), U17.14 (SCLK)
- net SDA: now also J20.5 (TP_SDA), U30.5 (SDA2); no longer J20.10 (TP_SDA), U15.25 (IO19), U17.13 (SDA)
- net SD_CD: no longer U15.56 (IO46)
- net SD_CLK: now also U15.24 (IO39); no longer U15.31 (SD_CLK)
- net SD_CMD: now also U15.25 (IO40); no longer U15.32 (SD_CMD)
- net SD_D0: now also U15.12 (IO35); no longer U15.27 (SD_D0)
- net SD_D1: now also U15.21 (IO36); no longer U15.28 (SD_D1)
- net SD_D2: now also U15.22 (IO37); no longer U15.29 (SD_D2)
- net SD_D3: now also U15.23 (IO38); no longer U15.30 (SD_D3)
- net SD_VDD_EN: no longer U15.57 (IO47)
- net SYS_POWER: now also U17.26 (VP), U4.6 (IN), C253.1, C254.1, R245.1; no longer U4.1 (IN)
- net SYS_PWR_EN: no longer U15.7 (IO3)
- net TP_INT: now also J20.7 (TP_INT); no longer J20.12 (TP_INT), U15.54 (IO44)
- net TP_RST: now also J20.9 (TP_RESET); no longer J20.14 (TP_RST)
- net TUSB_ID: no longer U15.22 (IO16)
- net TUSB_INT: no longer U15.20 (IO14)
- net UART_RX0: now also U15.36 (RX0); no longer U15.69 (RX0)
- net UART_TX0: now also U15.37 (TX0); no longer U15.68 (TX0)
- net C17_Pad2 renamed HPOUTA
- net C19_Pad2 renamed HPOUTB
- net DAC_BCK renamed FLYPVA
- removed net DAC_DATA: U15.66 (IO56), U17.8 (DACDAT)
- net DAC_LRCK renamed NVA
- net DAC_MCK renamed FLYNVA
- net JACK_DETECT renamed HPREFB
- net MCK_OSC renamed XTAL2
- net U17_CPCA renamed FILTP
- net U17_CPVOUTN renamed I2S_DIN_1V8
- net U17_LINEVOUTL renamed DAC_SCL
- net U17_LINEVOUTR renamed FLYNVCP
- net U17_VMID renamed VCPFN
- new net: U4.2 (NC), U4.5 (NC)
- new net: U34.2 (NC), U34.5 (NC)
- new net DAC_INT: R246.2, U17.27 (INT)
- new net DAC_RESET: Q20.1 (G), R244.2
- new net DAC_RESET_N: Q20.3 (D), R245.2, U17.28 (RESET)
- new net DAC_SDA: R248.2, U17.39 (SDA), U30.4 (SDA1)
- new net FILTN: C246.1, U17.6 (FILT-)
- new net FLYCVCP: C251.2, C252.1, U17.23 (FLYC_VCP)
- new net FLYPVCP: C251.1, U17.24 (FLYP_VCP)
- new net HPREFA: J1.1 (SLEEVE), U17.13 (HPREFA)
- new net HP_DETECT: J1.5 (TIP_SW), U17.22 (HP_DETECT)
- new net I2S_BCLK: U31.4 (B)
- new net I2S_BCLK_1V8: U17.34 (SCLK1), U31.3 (A)
- new net I2S_DOUT: U33.4 (B)
- new net I2S_LRCK: U32.4 (B)
- new net I2S_LRCK_1V8: U17.38 (LRCK1), U32.3 (A)
- new net PCA_EN: R247.2, U30.8 (EN)
- new net V1P8: C240.1, C241.1, C261.1, C262.1, FB1.1, R248.1, R249.1, U17.31 (VL), U17.4 (VD), U30.2 (VREF1), U31.1 (VCCA), U31.5 (DIR)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
- new net VCPFP: C249.1, U17.21 (VCP_FILT+)
- new net XTAL1: R240.1, X1.1
- new net XTAL3: R242.1, X2.1
- new net XTAL4: R243.1, X2.3
- new net XTI: C255.1, R240.2, R242.2, U17.37 (XTI/MCLK)
- new net XTO: C256.1, R241.2, R243.2, U17.36 (XTO)
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Other:
- note added: "AMOLED 2,06 Zoll 410 x 502 (CO5300, QSPI): FPC 30 Pol, Belegung wie Waveshare ESP32-S3-Touch-AMOLED-2.06"
- note added: "Audio: CS43131 (22,5792-MHz-Quarz, I2S-Master), 1,8-V-LDO, Pegelwandler, Klinke SJ-43504 + ESD (Tangara)"
- note added: "ESP32-S31-WROOM-1 (Espressif-Beschaltung)"
- note added: "Klickrad-Anschluss (FFC 6 Pol 0,5 mm), Befestigungsloecher M1,6"
- note removed: "AMOLED-Anschluss (FPC 34 Pol, wie Waveshare ESP32-S3-Touch-AMOLED-1.8)"
- note removed: "Audio: WM8523 + INA1620 + TPS65133 + Klinke (1:1 von Tangara, + MCLK-Option)"
- note removed: "ESP32-S31-WROOM-3 (Espressif-Beschaltung)"
- note removed: "Klickrad-Anschluss (JST-SH 6 Pol), Montagelocher"
- title: Hauptplatine Nano-Player (Endgeraet), Rev. 1 -> Hauptplatine Nano-Player (Endgeraet), Rev. 2

Commit message: Hauptplatine und S31-Test: Zwischenstand (in Arbeit)
Co-Authored-By: Claude Sonnet 5.5 <noreply@anthropic.com>
Claude-Session: https://claude.ai/code/session_01JifvE6gExGmwsJWDpfRrrS
Parts:
- removed H4: M1.6, Hauptplatine:MountingHole_1.8mm, symbol Mechanical:MountingHole
- added NT1: NetTie, NetTie:NetTie-2_SMD_Pad0.5mm, symbol Hauptplatine:NT1
- added NT2: NetTie, NetTie:NetTie-2_SMD_Pad0.5mm, symbol Hauptplatine:NT2
Connections:
- net CHG_PG: now also U15.30 (IO44)
- net CHG_PROG2: now also U15.32 (IO46)
- net CHG_SEL: now also U15.35 (IO55)
- net CHG_STAT1: now also U15.31 (IO45)
- net CHG_STAT2: now also U15.33 (IO47)
- net DAC_INT: now also U15.56 (IO48)
- net DAC_RESET: now also U15.17 (IO22)
- net FG_ALRT: now also U15.29 (IO43)
- net GND: now also NT1.2 (GND), NT2.2 (GND)
- net HOST_EN: now also U15.19 (IO24)
- net HPREFA: now also NT1.1 (REF)
- net HPREFB: now also NT2.1 (REF)
- net I2S_BCLK: now also U15.44 (IO10)
- net I2S_DOUT: now also U15.51 (IO17)
- net I2S_LRCK: now also U15.53 (IO19)
- net KEY_LOCK_MCU: now also U15.10 (IO6)
- net LCD_CS: now also U15.61 (IO53)
- net LCD_D0: now also U15.57 (IO49)
- net LCD_D1: now also U15.58 (IO50)
- net LCD_D2: now also U15.59 (IO51)
- net LCD_D3: now also U15.43 (IO9)
- net LCD_RST: now also U15.18 (IO23)
- net LCD_SCK: now also U15.42 (IO8)
- net LCD_TE: now also U15.52 (IO18)
- net SCL: now also U15.20 (IO25)
- net SDA: now also U15.28 (IO42)
- net SD_CD: now also U15.38 (IO56)
- net SD_VDD_EN: now also U15.34 (IO54)
- net SYS_PWR_EN: now also U15.9 (IO1)
- net TP_INT: now also U15.60 (IO52)
- net TUSB_ID: now also U15.16 (IO21)
- net TUSB_INT: now also U15.15 (IO20)
- net WHEEL_INT: now also U15.11 (IO7)
- new net: U15.26 (NC), U15.39 (NC), U15.4 (NC), U15.45 (NC), U15.46 (NC), U15.47 (NC), U15.48 (NC), U15.49 (NC), U15.5 (NC), U15.50 (NC), U15.6 (NC), U15.7 (NC), U15.8 (NC)

Commit message: Hauptplatine geroutet: Doku, Maße und Problemliste aktualisiert
Co-Authored-By: Claude Sonnet 5.5 <noreply@anthropic.com>
Claude-Session: https://claude.ai/code/session_01JifvE6gExGmwsJWDpfRrrS
Parts:
- J21: value FH12-6S-0.5SH(55) -> 503480-0600; footprint Connector_FFC-FPC:Hirose_FH12-6S-0.5SH_1x06-1MP_P0.50mm_Horizontal -> Hauptplatine:Molex_503480-0600; Beschreibung Klickrad-Modul v2 (AT42QT2120 0x1C + DRV2605L 0x5A), gleich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 -> Klickrad-Stecker Molex 503480-0600 (Easy-On BackFlip, Dual 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; DigiKey (none) -> WM1387CT-ND; Hersteller Hirose -> Molex; MPN FH12-6S-0.5SH(55) -> 503480-0600
Connections:
- net CHG_PG: now also U15.51 (IO17); no longer U15.30 (IO44)
- net CHG_PROG2: now also U15.48 (IO14); no longer U15.32 (IO46)
- net CHG_SEL: now also U15.49 (IO15); no longer U15.35 (IO55)
- net CHG_STAT1: now also U15.47 (IO13); no longer U15.31 (IO45)
- net CHG_STAT2: now also U15.50 (IO16); no longer U15.33 (IO47)
- net DAC_INT: now also U15.16 (IO21); no longer U15.56 (IO48)
- net DAC_RESET: now also U15.15 (IO20); no longer U15.17 (IO22)
- net FG_ALRT: now also U15.9 (IO1); no longer U15.29 (IO43)
- net HOST_EN: now also U15.4 (IO2); no longer U15.19 (IO24)
- net I2S_BCLK: now also U15.17 (IO22); no longer U15.44 (IO10)
- net I2S_DOUT: now also U15.19 (IO24); no longer U15.51 (IO17)
- net I2S_LRCK: now also U15.18 (IO23); no longer U15.53 (IO19)
- net KEY_LOCK_MCU: now also U15.7 (IO5); no longer U15.10 (IO6)
- net LCD_CS: now also U15.57 (IO49); no longer U15.61 (IO53)
- net LCD_D0: now also U15.45 (IO11); no longer U15.57 (IO49)
- net LCD_D1: now also U15.44 (IO10); no longer U15.58 (IO50)
- net LCD_D2: now also U15.43 (IO9); no longer U15.59 (IO51)
- net LCD_D3: now also U15.59 (IO51); no longer U15.43 (IO9)
- net LCD_RST: now also U15.53 (IO19); no longer U15.18 (IO23)
- net LCD_SCK: now also U15.56 (IO48); no longer U15.42 (IO8)
- net LCD_TE: now also U15.46 (IO12); no longer U15.52 (IO18)
- net SCL: now also U15.11 (IO7); no longer U15.20 (IO25)
- net SDA: now also U15.10 (IO6); no longer U15.28 (IO42)
- net SD_CD: now also U15.20 (IO25); no longer U15.38 (IO56)
- net SD_VDD_EN: now also U15.28 (IO42); no longer U15.34 (IO54)
- net SYS_PWR_EN: now also U15.6 (IO4); no longer U15.9 (IO1)
- net TP_INT: now also U15.58 (IO50); no longer U15.60 (IO52)
- net TUSB_ID: now also U15.5 (IO3); no longer U15.16 (IO21)
- net TUSB_INT: now also U15.52 (IO18); no longer U15.15 (IO20)
- net WHEEL_INT: now also U15.8 (IO0); no longer U15.11 (IO7)
- net at U4.2 (NC_2): no longer U4.5 (NC)
- net at U34.2 (NC_2): no longer U34.5 (NC)
- net at J6.A8 (NC_A8): no longer J6.B8 (NC)
- now unconnected: U15.26 (NC), U15.39 (NC), U17.12 (NC), U17.15 (NC), U17.29 (NC), U17.3 (NC), U17.32 (NC), U17.33 (NC), U17.40 (NC)
- no-connect marks 11 -> 32

Commit message: Hauptplatine Rev. 3b: Review-Fixes (B1-B3, H1, H4, H5, H7, H8), Doku
Co-Authored-By: Claude Sonnet 5.5 <noreply@anthropic.com>
Claude-Session: https://claude.ai/code/session_01JifvE6gExGmwsJWDpfRrrS
Parts:
- added Q21, Q22: 2N7002T, Package_TO_SOT_SMD:SOT-523, symbol Hauptplatine:Q_NMOS_123
- added R250: 100k, Resistor_SMD:R_0402_1005Metric, symbol Device:R
- added SW2, SW3: B3U-3000P, Button_Switch_SMD:SW_SPST_B3U-3000P, symbol Switch:SW_Push
- C257: value 100nF -> 100pF; Beschreibung PCA9306 VREF2 -> PCA9306 VREF2/EN nach GND (100 pF, Review B1); Hersteller Samsung -> Murata; LCSC C1525 -> (none); MPN CL05B104KO5NNNC -> GRM1555C1H101JA01D
- J20: value FH12-30S-0.5SH(55) -> 503480-3000; footprint Connector_FFC-FPC:Hirose_FH12-30S-0.5SH_1x30-1MP_P0.50mm_Horizontal -> Hauptplatine:Molex_503480-3000; Beschreibung Display-FPC-Stecker, 30 Pin 0,5 mm (Waveshare 2,06'-Board J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 -> Display-FPC-Stecker, 30 Pin 0,5 mm, Molex Easy-On BackFlip,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; DigiKey (none) -> 5034803000 (Digi-Key-Artikelseite 15710893); Hersteller Hirose -> Molex; MPN FH12-30S-0.5SH(55) -> 5034803000
- R1: Beschreibung (none) -> NUR bestuecken, wenn die Zelle KEINEN eigenen 10-k-NTC hat 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; Herkunft Tangara -> angepasst; now not fitted
- R247: Beschreibung EN-Pull-up PCA9306 (200 k laut Datenblatt) -> VREF2/EN-Pull-up PCA9306 (200 k laut Datenblatt, gemeinsame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; Hersteller (none) -> UNI-ROYAL; MPN (none) -> 0402WGF2003TCE
- R36: Beschreibung PROG2 hoch = USB-Eingangslimit 500 mA (Tangara: Pin vom SAM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 -> PROG2 fest hoch = USB-Eingangslimit 500 mA (SEL = GND, USB-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
- R39: value 1k -> 2.7k; Beschreibung (none) -> PROG1 2,7 k = ca. 370 mA Ladestrom (1000 V / R) fuer eine Z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; Herkunft Tangara -> angepasst; MPN RC0603DR-071KL -> AC0603FR-072K7L
- R43: Beschreibung SEL hoch = USB-Eingang (Tangara Rev. 4) -> SEL fest nach GND = USB-Modus (SEL hoch waere AC-Adapter-Mo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
- R57: Beschreibung (none) -> NICHT bestuecken: IO36 ist Strapping-Pin (VDD_SPI), SD_VDD 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; Herkunft Tangara -> angepasst; now not fitted
- U30: Beschreibung I2C-Pegelwandler 1,8 V (DAC) <-> 3,3 V (Bus); EN ueber 200 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 -> I2C-Pegelwandler 1,8 V (DAC) <-> 3,3 V (Bus); VREF2 (Pin 7)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
Connections:
- net 3V3: now also Q22.1 (G); no longer C257.1, R36.1, R43.1, U30.7 (VREF2)
- net BOOT: now also SW2.1
- net CHG_PROG2: no longer U15.48 (IO14)
- net CHG_SEL: no longer U15.49 (IO15)
- net DAC_RESET_N: now also Q21.3 (D)
- net ESP_EN: now also SW3.1
- net GND: now also R43.1, Q21.2 (S), Q22.2 (S), SW2.2, SW3.2
- net PCA_EN: now also C257.1, U30.7 (VREF2)
- net SYS_POWER: now also R250.1
- net VBUS_SW: now also R36.1
- new net RST_G: Q21.1 (G), Q22.3 (D), R250.2
- no-connect marks 32 -> 34
Other:
- title: Hauptplatine Nano-Player (Endgeraet), Rev. 2 -> Hauptplatine Nano-Player (Endgeraet), Rev. 3b
