File: hardware/pcb/klickrad/klickrad.kicad_pcb (KiCad board)
At the start: 2 copper layers, 32 x 32 mm, 24 parts, among them J1 503480-0600, SW1 BUTTON, SW2 WHEEL, SW3 GUARD, U1 AT42QT2120, U2 DRV2605LDGSR

Commit message: Klickrad J1 auf J21-Landmuster, neu geroutet; TEILE-Nachtrag
Co-Authored-By: Claude Sonnet 5.5 <noreply@anthropic.com>
Claude-Session: https://claude.ai/code/session_01JifvE6gExGmwsJWDpfRrrS
Parts:
- J1: footprint Klickrad:Molex_503480-0600_1x06-1MP_P0.50mm_Horizontal -> Klickrad:Molex_503480-0600_Hauptplatine
- turned J1 to 0 degrees
Routing:
- net 3V3: track 43.7 -> 57.3 mm, vias 2 -> 4
- net SDA: track 14.6 -> 18.2 mm, vias 3 -> 2
- net SCL: track 21.8 -> 25.1 mm
- net E0: track 14.1 -> 16.1 mm
- net CHANGE: track 9.75 -> 11.7 mm
- net EG: track 12.6 -> 11.5 mm
- net LRA_P: track 2.72 -> 3.64 mm
- net GND: track 32.2 -> 31.6 mm
Other:
- board text added: "I2C 1C/5A"
- board text added: "LRA max 14x6x3"
- board text removed: "(6)"
- board text removed: "3V3"
- board text removed: "CHG"
- board text removed: "GND"
- board text removed: "LRA bis 3 mm hoch: 12x6 / 16x6"
- board text removed: "QT2120 0x1C DRV 0x5A"
- board text removed: "SCL"
- board text removed: "SDA"
